File: kicad/gdl90_2_g496.sch (KiCad schematic (older format))
At the start: 1 part

Commit message: ESP32 adaptation
Parts:
- added J1: DB9_Male, Connector_Dsub:DSUB-9_Male_Horizontal_P2.77x2.84mm_EdgePinOffset4.94mm_Housed_MountingHolesOffset7.48mm, symbol Connector:DB9_Male
- added R1: 10K, Resistor_SMD:R_0805_2012Metric, symbol Device:R
- added U1: MAX233CPP, max233:MAX233CPP, symbol 2020-10-19_23-45-47:MAX233CPP
- added U2, U3: LM2937xMP, Package_TO_SOT_SMD:SOT-223-3_TabPin2, symbol Regulator_Linear:LM2937xMP
- added U?: ESP32-WROVER, symbol esp32-wrover:ESP32-WROVER
- U4: renamed from U?; footprint (none) -> nodemcu:NodeMCU_0.9; symbol ESP8266:NodeMCU1.0(ESP-12E) -> gdl90_2_g496-rescue:NodeMCU1.0(ESP-12E)-ESP8266
Connections:
- net GND: now reaches U4.10 (GND)
- net GND: now also U4.14 (GND), U4.17 (GND), U4.24 (GND), J1.6, R1.2, U1.6 (GND), U1.9 (GND), U2.2 (GND), U3.2 (GND)
- net +3V3: now reaches U4.11 (3.3V)
- net +3V3: now also U4.16 (3.3V), U4.25 (3.3V), J1.8, U2.3 (VO)
- net at U4.21 (D7(GPIO13)): now also U1.3 (R1_OUT)
- net at U4.26 (D4(GPIO2)): now also U1.2 (T1_IN)
- net at U4.28 (D2(GPIO4)): now also J1.4, R1.1
- new net: U1.10 (C2-), U1.16 (C2-)
- new net: U1.11 (C2+), U1.15 (C2+)
- new net: U1.12 (V-), U1.17 (V-)
- new net: J1.9, U1.4 (R1_IN)
- new net: J1.5, U1.5 (T1_OUT)
- new net +12V: J1.1, U2.1 (VI), U3.1 (VI)
- new net +5V: U1.7 (VCC), U3.3 (VO)
- no-connect marks 0 -> 32
